File: flex/flex.kicad_pcb (KiCad board)
At the start: 2 copper layers, 126.3 x 90.6 mm, 85 parts, among them J1 Conn_01x04_Female, J2 Conn_01x05_Female, J3 Conn_01x03_Female, J4 Conn_01x06_Female, J5 Conn_01x03_Female, SW10 SW_Push, SW11 SW_Push, SW12 SW_Push, SW15 SW_Push, SW16 SW_Push, SW17 SW_Push, SW2 SW_Push, SW20 SW_Push, SW21 SW_Push, SW22 SW_Push, SW24 SW_Push, SW25 SW_Push, SW26 SW_Push, SW3 SW_Push, SW4 SW_Push, SW6 SW_Push, SW7 SW_Push, SW8 SW_Push

Commit message: edge cuts
Parts:
- added SW10: SW_Push, custom:SW_MX_reversible, B.Cu at (87.3, 66.3)
- added SW11: SW_Push, custom:SW_MX_reversible, B.Cu at (87.3, 89.2)
- added SW12: SW_Push, custom:SW_MX_reversible, B.Cu at (87.3, 112.2)
- added SW15: SW_Push, custom:SW_MX_reversible, B.Cu at (109.2, 64.0)
- added SW16: SW_Push, custom:SW_MX_reversible, B.Cu at (109.2, 87.0)
- added SW17: SW_Push, custom:SW_MX_reversible, B.Cu at (109.2, 109.9)
- C1, C2: value C -> 1u
- R1, R2: value R -> 330
- moved C2 157.4 mm to (-105.8, 68.7)
- moved D10 157.4 mm to (-120.5, 105.1)
- moved D11 157.4 mm to (-76.8, 68.1)
- moved D12 157.4 mm to (-98.1, 112.6)
- moved D13 157.4 mm to (-54.3, 65.8)
- moved D15 157.4 mm to (-98.3, 105.1)
- moved D19 157.4 mm to (-76.3, 90.4)
- moved D27 157.4 mm to (-54.1, 88.5)
- moved G*** 157.4 mm to (-104.2, 51.5)
- moved J3 157.4 mm to (-103.5, 67.3)
- moved R1 157.4 mm to (-107.6, 76.2)
- moved SW10 157.4 mm to (-69.9, 58.5)
- moved SW11 157.4 mm to (-69.9, 81.4)
- moved SW12 157.4 mm to (-69.9, 104.4)
- moved SW15 157.4 mm to (-48.0, 56.3)
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Connections:
- J2 pad 2: Net-(J2-Pad2) -> unconnected-(J2-Pin_2-Pad2)
Routing:
- net (no net): track 0.00 -> 651.8 mm, vias 0 -> 24
- net Net-(D25-DOUT): track 127.8 -> 0.00 mm, vias 2 -> 0
- net Net-(D18-DOUT): track 124.7 -> 0.00 mm, vias 2 -> 0
- net Net-(D21-DIN): track 120.4 -> 0.00 mm, vias 4 -> 0
- net Net-(D33-DIN): track 45.7 -> 0.00 mm, vias 3 -> 0
- net Net-(D21-DOUT): track 45.1 -> 0.00 mm, vias 4 -> 0
- net Net-(D28-DOUT): track 44.1 -> 0.00 mm, vias 2 -> 0
- net Net-(D18-DIN): track 41.4 -> 0.00 mm, vias 2 -> 0
- net Net-(D5-DOUT): track 40.3 -> 0.00 mm, vias 2 -> 0
- net Net-(D23-DOUT): track 38.2 -> 0.00 mm, vias 2 -> 0
- net Net-(D37-DOUT): track 38.3 -> 22.4 mm, vias 2 -> 1
- net Net-(D39-DOUT): track 47.2 -> 39.0 mm
Other:
- board size 126.3 x 90.6 mm -> 126.3 x 91.6 mm

Commit message: place components
Parts:
- moved D1 165.5 mm to (45.1, 111.8)
- moved D10 162.1 mm to (41.6, 111.8)
- moved D11 157.5 mm to (80.7, 70.5)
- moved R1 157.4 mm to (49.6, 83.0)
- moved R2 157.4 mm to (49.6, 83.0)
- moved D17 157.4 mm to (80.8, 116.7)
- moved D9 157.3 mm to (58.8, 82.9)
- moved D2 157.2 mm to (37.4, 83.5)
- moved D20 157.2 mm to (102.8, 114.5)
- moved D15 157.1 mm to (58.8, 105.8)
- moved D13 157.1 mm to (102.8, 68.3)
- moved D19 157.0 mm to (80.7, 93.9)
- moved C2 156.9 mm to (51.0, 75.6)
- moved J3 156.9 mm to (53.3, 74.2)
- moved C1 156.9 mm to (51.0, 75.6)
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Routing:
- net Vcc: track 702.6 -> 0.00 mm, vias 19 -> 0
- net Gnd: track 699.9 -> 0.00 mm, vias 27 -> 0
- net (no net): track 651.8 -> 0.00 mm, vias 24 -> 0
- net row2: track 481.4 -> 0.00 mm, vias 5 -> 0
- net row4: track 431.6 -> 0.00 mm, vias 7 -> 0
- net col1: track 278.4 -> 0.00 mm, vias 6 -> 0
- net row3: track 265.4 -> 0.00 mm, vias 3 -> 0
- net col2: track 256.2 -> 0.00 mm, vias 10 -> 0
- net col6: track 174.7 -> 0.00 mm, vias 7 -> 0
- net col5: track 158.5 -> 0.00 mm, vias 6 -> 0
- net Net-(D41-DOUT): track 147.8 -> 0.00 mm, vias 3 -> 0
- net col3: track 143.7 -> 0.00 mm, vias 6 -> 0
- net col4: track 129.2 -> 0.00 mm, vias 5 -> 0
- net Net-(D51-DOUT): track 103.0 -> 0.00 mm, vias 3 -> 0
- net row5: track 43.1 -> 0.00 mm, vias 1 -> 0
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Other:
- outline, holes or cut-outs redrawn

Commit message: routing
Routing:
- net Gnd: track 0.00 -> 754.7 mm, vias 0 -> 18
- net Vcc: track 0.00 -> 725.8 mm, vias 0 -> 18
- net col1: track 0.00 -> 265.9 mm, vias 0 -> 5
- net col2: track 0.00 -> 227.6 mm, vias 0 -> 4
- net col3: track 0.00 -> 146.7 mm, vias 0 -> 3
- net col4: track 0.00 -> 87.0 mm, vias 0 -> 2
- net Din: track 0.00 -> 7.91 mm, vias 0 -> 1
- net Net-(D28-DIN): track 0.00 -> 2.57 mm, vias 0 -> 1
- net Net-(D9-A): track 0.00 -> 1.92 mm
- net Net-(D27-A): track 0.00 -> 1.92 mm
- net Net-(D20-A): track 0.00 -> 1.92 mm
- net Net-(D2-A): track 0.00 -> 1.92 mm
- net Net-(D19-A): track 0.00 -> 1.92 mm
- net Net-(D15-A): track 0.00 -> 1.92 mm
- net Net-(D13-A): track 0.00 -> 1.92 mm
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- added copper zone on B.Cu, net Gnd
- added copper zone on F.Cu, net Gnd

Commit message: routing
Routing:
- net col6: track 0.00 -> 5.75 mm
- net col5: track 0.00 -> 5.75 mm
- net Net-(D36-A): track 0.00 -> 1.92 mm
- net Net-(D35-A): track 0.00 -> 1.92 mm
- net Net-(D32-A): track 0.00 -> 1.92 mm
- net Net-(D31-A): track 0.00 -> 1.92 mm
- net Net-(D16-A): track 0.00 -> 1.92 mm
- net Net-(D14-A): track 0.00 -> 1.92 mm
Changed lines of the file:
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@@
-	)
-	(segment
-		(start 101.25 114.05)
-		(end 102.65 115.45)
-		(width 0.13)
-		(layer "B.Cu")
-		(net 9)
 	)
 	(segment
@@
 	)
 	(segment
-		(start 103.5 108.9)
-		(end 101.25 111.15)
-		(width 0.13)
-		(layer "B.Cu")
-		(net 9)
-	)
-	(segment
 		(start 115.6 74.57168)
 		(end 115.6 75.6)
@@
 	)
 	(segment
+		(start 102.35 115.45)
+		(end 103.65 115.45)
+		(width 0.13)
+		(layer "B.Cu")
+		(net 9)
+	)
+	(segment
+		(start 103.5 108.9)
+		(end 101.4 111)
+		(width 0.13)
+		(layer "B.Cu")
+		(net 9)
+	)
+	(segment
+		(start 104.65 79.6)
+		(end 114.9 79.6)
+		(width 0.13)
+		(layer "B.Cu")
+		(net 9)
+	)
+	(segment
+		(start 101.4 111)
+		(end 101.4 114.5)
+		(width 0.13)
+		(layer "B.Cu")
+		(net 9)
+	)
+	(segment
 		(start 103.5 93.2)
 		(end 103.5 108.9)
@@
 	)
 	(segment
-		(start 104.65 79.6)
-		(end 114.9 79.6)
-		(width 0.13)
-		(layer "B.Cu")
-		(net 9)
-	)
-	(segment
-		(start 101.25 111.15)
-		(end 101.25 114.05)
-		(width 0.13)
-		(layer "B.Cu")
-		(net 9)
-	)
-	(segment
-		(start 102.65 115.45)
-		(end 103.65 115.45)
-		(width 0.13)
-		(layer "B.Cu")
-		(net 9)
-	)
-	(segment
 		(start 114.9 79.6)
 		(end 115.825735 78.674265)
@@
 		(layer "B.Cu")
 		(net 9)
+	)
+	(segment
+		(start 101.4 114.5)
+		(end 102.35 115.45)
+		(width 0.13)
+		(layer "B.Cu")
+		(net 9)
+	)
+	(segment
+		(start 125.8252 120.2105)
+		(end 125.8252 119.25275)
+		(width 0.13)
+		(layer "F.Cu")
+		(net 13)
+	)
+	(segment
+		(start 126.3752 73.80275)
+		(end 126.3752 74.7605)
+		(width 0.13)
+		(layer "F.Cu")
+		(net 13)
+	)
+	(segment
+		(start 126.3752 97.1605)
+		(end 126.3752 96.20275)
+		(width 0.13)
+		(layer "F.Cu")
+		(net 13)
+	)
+	(segment
+		(start 125.8252 120.2105)
+		(end 125.8252 119.25275)
+		(width 0.13)
+		(layer "B.Cu")
+		(net 13)
+	)
+	(segment
+		(start 126.3752 73.80275)
+		(end 126.3752 74.7605)
+		(width 0.13)
+		(layer "B.Cu")
+		(net 13)
+	)
+	(segment
+		(start 126.3752 96.20275)
+		(end 126.3752 97.1605)
+		(width 0.13)
+		(layer "B.Cu")
+		(net 13)
+	)
+	(segment
+		(start 147.65 74.15775)
+		(end 147.65 73.2)
+		(width 0.13)
+		(layer "F.Cu")
+		(net 14)
+	)
+	(segment
+		(start 152.4252 104.6105)
+		(end 152.4252 103.65275)
+		(width 0.13)
+		(layer "F.Cu")
+		(net 14)
+	)
+	(segment
+		(start 156.1752 104.6105)
+		(end 156.1752 103.65275)
+		(width 0.13)
+		(layer "F.Cu")
+		(net 14)
+	)
+	(segment
+		(start 156.1752 104.6105)
+		(end 156.1752 103.65275)
+		(width 0.13)
+		(layer "B.Cu")
+		(net 14)
+	)
+	(segment
+		(start 152.4252 103.65275)
+		(end 152.4252 104.6105)
+		(width 0.13)
+		(layer "B.Cu")
+		(net 14)
+	)
+	(segment
+		(start 147.65 73.2)
+		(end 147.65 74.15775)
+		(width 0.13)
+		(layer "B.Cu")
+		(net 14)
 	)
 	(segment
@@
 	)
 	(segment
+		(start 126.3752 71.70275)
+		(end 126.3752 70.745)
+		(width 0.13)
+		(layer "F.Cu")
+		(net 25)
+	)
+	(segment
+		(start 126.3752 70.745)
+		(end 126.3752 71.70275)
+		(width 0.13)
+		(layer "B.Cu")
+		(net 25)
+	)
+	(segment
 		(start 58.8 104.7)
 		(end 58.8 103.74225)
@@
 	)
 	(segment
+		(start 147.65 71.1)
+		(end 147.65 70.14225)
+		(width 0.13)
+		(layer "F.Cu")
+		(net 27)
+	)
+	(segment
+		(start 147.65 70.14225)
+		(end 147.65 71.1)
+		(width 0.13)
+		(layer "B.Cu")
+		(net 27)
+	)
+	(segment
 		(start 80.75 115.6)
 		(end 80.75 114.64225)
@@
 	)
 	(segment
+		(start 125.8252 117.15275)
+		(end 125.8252 116.195)
+		(width 0.13)
+		(layer "F.Cu")
+		(net 36)
+	)
+	(segment
+		(start 125.8252 117.15275)
+		(end 125.8252 116.195)
+		(width 0.13)
+		(layer "B.Cu")
+		(net 36)
+	)
+	(segment
+		(start 126.3752 94.10275)
+		(end 126.3752 93.145)
+		(width 0.13)
+		(layer "F.Cu")
+		(net 37)
+	)
+	(segment
+		(start 126.3752 93.145)
+		(end 126.3752 94.10275)
+		(width 0.13)
+		(layer "B.Cu")
+		(net 37)
+	)
+	(segment
+		(start 156.1752 101.55275)
+		(end 156.1752 100.595)
+		(width 0.13)
+		(layer "F.Cu")
+		(net 38)
+	)
+	(segment
+		(start 156.1752 101.55275)
+		(end 156.1752 100.595)
+		(width 0.13)
+		(layer "B.Cu")
+		(net 38)
+	)
+	(segment
+		(start 152.4252 101.55275)
+		(end 152.4252 100.595)
+		(width 0.13)
+		(layer "F.Cu")
+		(net 39)
+	)
+	(segment
+		(start 152.4252 100.595)
+		(end 152.4252 101.55275)
+		(width 0.13)
+		(layer "B.Cu")
+		(net 39)
+	)
+	(segment
