File: flex/flex.kicad_pcb (KiCad board)
At the start: 2 copper layers, 126.3 x 90.6 mm, 85 parts, among them J1 Conn_01x04_Female, J2 Conn_01x05_Female, J3 Conn_01x03_Female, J4 Conn_01x06_Female, J5 Conn_01x03_Female, SW10 SW_Push, SW11 SW_Push, SW12 SW_Push, SW15 SW_Push, SW16 SW_Push, SW17 SW_Push, SW2 SW_Push, SW20 SW_Push, SW21 SW_Push, SW22 SW_Push, SW24 SW_Push, SW25 SW_Push, SW26 SW_Push, SW3 SW_Push, SW4 SW_Push, SW6 SW_Push, SW7 SW_Push, SW8 SW_Push

Commit message: jlc changes
Other:
- board text added: "Ergonomic keyboard innovation"
- board text added: "REV 2.22"
- board text removed: "Custom keyboards made in the Netherlands"
- board text removed: "REV 2.21"
