File: flex/flex.kicad_sch (KiCad schematic)
At the start: 81 parts, among them J1 Conn_01x04_Female, J2 Conn_01x05_Female, J3 Conn_01x03_Female, J4 Conn_01x06_Female, J5 Conn_01x03_Female, SW10 SW_Push, SW11 SW_Push, SW12 SW_Push, SW15 SW_Push, SW16 SW_Push, SW17 SW_Push, SW2 SW_Push, SW20 SW_Push, SW21 SW_Push, SW22 SW_Push, SW24 SW_Push, SW25 SW_Push, SW26 SW_Push, SW3 SW_Push, SW4 SW_Push, SW6 SW_Push, SW7 SW_Push, SW8 SW_Push

Commit message: rgb leds gnd silkscreen
Parts:
- D18, D21, D23, D25, D3, D33, D37, D39, D4, D41, D47, D49, D5, D51, D55, D57, D59, D7: footprint libs2:YS-SK6812MINI-E_REVERSE -> custom:SK6812_mini_e_corners
- D22, D24, D26, D28, D29, D30, D34, D38, D40, D42, D48, D50, D52, D56, D58, D6, D60, D8: footprint libs2:YS-SK6812MINI-E_REVERSE_NO_EDGECUT -> custom:SK6812_mini_e_corners_NOEDGECUTS
Changed lines of the file:
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@@
 			)
 		)
-		(property "Footprint" "libs2:YS-SK6812MINI-E_REVERSE_NO_EDGECUT"
+		(property "Footprint" "custom:SK6812_mini_e_corners_NOEDGECUTS"
 			(at 193.04 198.12 0)
 			(effects
@@
 			)
 		)
-		(property "Footprint" "libs2:YS-SK6812MINI-E_REVERSE_NO_EDGECUT"
+		(property "Footprint" "custom:SK6812_mini_e_corners_NOEDGECUTS"
 			(at 148.59 151.765 0)
 			(effects
@@
 			)
 		)
-		(property "Footprint" "libs2:YS-SK6812MINI-E_REVERSE"
+		(property "Footprint" "custom:SK6812_mini_e_corners"
 			(at 126.365 177.165 0)
 			(effects
@@
 			)
 		)
-		(property "Footprint" "libs2:YS-SK6812MINI-E_REVERSE"
+		(property "Footprint" "custom:SK6812_mini_e_corners"
 			(at 223.52 130.81 0)
 			(effects
@@
 			)
 		)
-		(property "Footprint" "libs2:YS-SK6812MINI-E_REVERSE"
+		(property "Footprint" "custom:SK6812_mini_e_corners"
 			(at 170.815 177.165 0)
 			(effects
@@
 			)
 		)
-		(property "Footprint" "libs2:YS-SK6812MINI-E_REVERSE"
+		(property "Footprint" "custom:SK6812_mini_e_corners"
 			(at 193.04 177.165 0)
 			(effects
@@
 			)
 		)
-		(property "Footprint" "libs2:YS-SK6812MINI-E_REVERSE"
+		(property "Footprint" "custom:SK6812_mini_e_corners"
 			(at 104.14 177.165 0)
 			(effects
@@
 			)
 		)
-		(property "Footprint" "libs2:YS-SK6812MINI-E_REVERSE_NO_EDGECUT"
+		(property "Footprint" "custom:SK6812_mini_e_corners_NOEDGECUTS"
 			(at 103.505 241.935 0)
 			(effects
@@
 			)
 		)
-		(property "Footprint" "libs2:YS-SK6812MINI-E_REVERSE"
+		(property "Footprint" "custom:SK6812_mini_e_corners"
 			(at 215.265 177.165 0)
 			(effects
@@
 			)
 		)
-		(property "Footprint" "libs2:YS-SK6812MINI-E_REVERSE"
+		(property "Footprint" "custom:SK6812_mini_e_corners"
 			(at 103.505 220.98 0)
 			(effects
@@
 			)
 		)
-		(property "Footprint" "libs2:YS-SK6812MINI-E_REVERSE_NO_EDGECUT"
+		(property "Footprint" "custom:SK6812_mini_e_corners_NOEDGECUTS"
 			(at 214.63 241.935 0)
 			(effects
@@
 			)
 		)
-		(property "Footprint" "libs2:YS-SK6812MINI-E_REVERSE_NO_EDGECUT"
+		(property "Footprint" "custom:SK6812_mini_e_corners_NOEDGECUTS"
 			(at 215.265 198.12 0)
 			(effects
@@
 			)
 		)
-		(property "Footprint" "libs2:YS-SK6812MINI-E_REVERSE"
+		(property "Footprint" "custom:SK6812_mini_e_corners"
 			(at 236.855 220.98 0)
 			(effects
@@
 			)
 		)
-		(property "Footprint" "libs2:YS-SK6812MINI-E_REVERSE_NO_EDGECUT"
+		(property "Footprint" "custom:SK6812_mini_e_corners_NOEDGECUTS"
 			(at 104.14 198.12 0)
 			(effects
@@
 			)
 		)
-		(property "Footprint" "libs2:YS-SK6812MINI-E_REVERSE_NO_EDGECUT"
+		(property "Footprint" "custom:SK6812_mini_e_corners_NOEDGECUTS"
 			(at 223.52 151.765 0)
 			(effects
@@
 			)
 		)
-		(property "Footprint" "libs2:YS-SK6812MINI-E_REVERSE_NO_EDGECUT"
+		(property "Footprint" "custom:SK6812_mini_e_corners_NOEDGECUTS"
 			(at 148.59 198.12 0)
 			(effects
@@
 			)
 		)
-		(property "Footprint" "libs2:YS-SK6812MINI-E_REVERSE"
+		(property "Footprint" "custom:SK6812_mini_e_corners"
 			(at 179.07 130.81 0)
 			(effects
@@
 			)
 		)
-		(property "Footprint" "libs2:YS-SK6812MINI-E_REVERSE"
+		(property "Footprint" "custom:SK6812_mini_e_corners"
 			(at 201.295 130.81 0)
 			(effects
@@
 			)
 		)
-		(property "Footprint" "libs2:YS-SK6812MINI-E_REVERSE_NO_EDGECUT"
+		(property "Footprint" "custom:SK6812_mini_e_corners_NOEDGECUTS"
 			(at 147.955 241.935 0)
 			(effects
@@
 			)
 		)
-		(property "Footprint" "libs2:YS-SK6812MINI-E_REVERSE_NO_EDGECUT"
+		(property "Footprint" "custom:SK6812_mini_e_corners_NOEDGECUTS"
 			(at 125.73 241.935 0)
 			(effects
@@
 			)
 		)
-		(property "Footprint" "libs2:YS-SK6812MINI-E_REVERSE_NO_EDGECUT"
+		(property "Footprint" "custom:SK6812_mini_e_corners_NOEDGECUTS"
 			(at 236.855 241.935 0)
 			(effects
@@
 			)
 		)
-		(property "Footprint" "libs2:YS-SK6812MINI-E_REVERSE"
+		(property "Footprint" "custom:SK6812_mini_e_corners"
 			(at 214.63 220.98 0)
 			(effects
@@
 			)
 		)
-		(property "Footprint" "libs2:YS-SK6812MINI-E_REVERSE_NO_EDGECUT"
+		(property "Footprint" "custom:SK6812_mini_e_corners_NOEDGECUTS"
 			(at 192.405 241.935 0)
 			(effects
@@
 			)
 		)
-		(property "Footprint" "libs2:YS-SK6812MINI-E_REVERSE"
+		(property "Footprint" "custom:SK6812_mini_e_corners"
 			(at 148.59 177.165 0)
 			(effects
@@
 			)
 		)
-		(property "Footprint" "libs2:YS-SK6812MINI-E_REVERSE"
+		(property "Footprint" "custom:SK6812_mini_e_corners"
 			(at 125.73 220.98 0)
 			(effects
@@
 			)
 		)
-		(property "Footprint" "libs2:YS-SK6812MINI-E_REVERSE_NO_EDGECUT"
+		(property "Footprint" "custom:SK6812_mini_e_corners_NOEDGECUTS"
 			(at 126.365 151.765 0)
 			(effects
@@
 			)
 		)
-		(property "Footprint" "libs2:YS-SK6812MINI-E_REVERSE_NO_EDGECUT"
+		(property "Footprint" "custom:SK6812_mini_e_corners_NOEDGECUTS"
 			(at 104.14 151.765 0)
 			(effects
@@
 			)
 		)
-		(property "Footprint" "libs2:YS-SK6812MINI-E_REVERSE_NO_EDGECUT"
+		(property "Footprint" "custom:SK6812_mini_e_corners_NOEDGECUTS"
 			(at 170.815 198.12 0)
 			(effects
@@
 			)
 		)
-		(property "Footprint" "libs2:YS-SK6812MINI-E_REVERSE_NO_EDGECUT"
+		(property "Footprint" "custom:SK6812_mini_e_corners_NOEDGECUTS"
 			(at 179.07 151.765 0)
 			(effects
@@
 			)
 		)
-		(property "Footprint" "libs2:YS-SK6812MINI-E_REVERSE"
+		(property "Footprint" "custom:SK6812_mini_e_corners"
 			(at 126.365 130.81 0)
 			(effects
@@
 			)
 		)
-		(property "Footprint" "libs2:YS-SK6812MINI-E_REVERSE"
+		(property "Footprint" "custom:SK6812_mini_e_corners"
 			(at 148.59 130.81 0)
 			(effects
@@
 			)
 		)
-		(property "Footprint" "libs2:YS-SK6812MINI-E_REVERSE_NO_EDGECUT"
+		(property "Footprint" "custom:SK6812_mini_e_corners_NOEDGECUTS"
 			(at 201.295 151.765 0)
 			(effects
@@
 			)
 		)
-		(property "Footprint" "libs2:YS-SK6812MINI-E_REVERSE_NO_EDGECUT"
+		(property "Footprint" "custom:SK6812_mini_e_corners_NOEDGECUTS"
 			(at 126.365 198.12 0)
 			(effects
@@
 			)
 		)
-		(property "Footprint" "libs2:YS-SK6812MINI-E_REVERSE"
+		(property "Footprint" "custom:SK6812_mini_e_corners"
 			(at 104.14 130.81 0)
 			(effects
@@
 			)
 		)
-		(property "Footprint" "libs2:YS-SK6812MINI-E_REVERSE"
+		(property "Footprint" "custom:SK6812_mini_e_corners"
 			(at 192.405 220.98 0)
 			(effects
@@
 			)
 		)
-		(property "Footprint" "libs2:YS-SK6812MINI-E_REVERSE"
+		(property "Footprint" "custom:SK6812_mini_e_corners"
 			(at 147.955 220.98 0)
 			(effects
